File: ui/tqfp-sandwich-ui.sch (EAGLE design)
At the start: 40 parts, among them U1 MCP1754X-XXXXX/C, U3 MCP1754X-XXXXX/C

Commit message: GPS fix, Add LM386 (thanks Kris SQ3PCA)
Parts:
- added C12: 47nF, SparkFun-Capacitors:47NF-0603-25V-5%
- added C13: 100nF, SparkFun-Capacitors:1.0NF/1000PF-0603-50V-10%
- added C15: 220 uF, rcl:CPOL-USC
- added C16: 10uF, SparkFun-Capacitors:10UF-POLAR-EIA3216-16V-10%(TANT)
- added IC2: LM386MM-1, linear:LM386MM-1
- added R5, R6: 0, SparkFun-Resistors:0OHM-0603-1/10W-5%
- added R9: 10, SparkFun-Resistors:10OHM-0603-1/10W-5%
- added VR1: 10k, SparkFun-Resistors:TRIMPOT-SMD-3MM-OPEN-1/10W-25%
- R1: value 3.3k -> 0
- R4: value 0 -> 3.3k
Connections:
- new net +12V: J2.7, J2.8, R5.2
- new net N$11: C15.+, IC2.OUT, R9.2
- new net N$21: IC2.GAIN@1, VR1.CW
- new net N$22: C16.+, VR1.WIPER
- new net N$23: C16.-, IC2.GAIN@2
- new net N$24: C13.2, IC2.VS, R5.1
- new net N$9: C12.1, R9.1
- new net SPK_AUDIO: C15.-, R24.2, R6.2
- net AUDIO: now also IC2.+IN, R6.1; no longer R24.2
- net GND: now also C12.2, C13.1, IC2.-IN, IC2.GND
- net N$3: now also R2.1, R4.2; no longer R4.1
- net PD0_RXD: no longer R2.1
- net PD1_TXD: now also R4.1; no longer R4.2
Other:
- note added: "AUDIO AMPLIFIER BYPASS"
- note added: "D"
- note removed: "C"
- moved on the sheet: ANT-CHIP, C1, C10, C2, C3, MIC, MIC., R1, R2, R3, R4, S4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
